Commit message: new icub urdfs and related meshes added

File: app/urdfs/iCubGenova02.urdf (robot description, URDF)
Before this commit: robot ICUB_2-5_BB_SIM_MODEL, 163 links, 162 joints
Links:
- link chest: mass 7.638 -> 5.638; geometry collision mesh filename=package://testbot_description/meshes/dae/sim_sea_2-5_chest_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 scale=0.001 0.001 0.001; visual mesh filename=package://testbot_description/meshes/dae/sim_sea_2-5_chest_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 scale=0.001 0.001 0.001
- link head: geometry collision mesh filename=package://testbot_description/meshes/dae/sim_sea_2-5_head_p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 scale=0.001 0.001 0.001; visual mesh filename=package://testbot_description/meshes/dae/sim_sea_2-5_head_p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 scale=0.001 0.001 0.001
- link l_ankle_1: geometry collision mesh filename=package://testbot_description/meshes/dae/sim_sea_2-5_l_ankl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 scale=0.001 0.001 0.001; visual mesh filename=package://testbot_description/meshes/dae/sim_sea_2-5_l_ankl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 scale=0.001 0.001 0.001
- link l_ankle_2: geometry collision mesh filename=package://testbot_description/meshes/dae/sim_sea_2-5_l_foot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 scale=0.001 0.001 0.001; visual mesh filename=package://testbot_description/meshes/dae/sim_sea_2-5_l_foot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 scale=0.001 0.001 0.001
- link l_elbow_1: geometry collision mesh filename=package://testbot_description/meshes/dae/sim_sea_2-5_l_elbo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 scale=0.001 0.001 0.001; visual mesh filename=package://testbot_description/meshes/dae/sim_sea_2-5_l_elbo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 scale=0.001 0.001 0.001
- link l_foot: geometry collision mesh filename=package://testbot_description/meshes/dae/sim_sea_2-5_l_sole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 scale=0.001 0.001 0.001; visual mesh filename=package://testbot_description/meshes/dae/sim_sea_2-5_l_sole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 scale=0.001 0.001 0.001
- link l_forearm: geometry collision mesh filename=package://testbot_description/meshes/dae/sim_sea_2-5_l_fore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 scale=0.001 0.001 0.001; visual mesh filename=package://testbot_description/meshes/dae/sim_sea_2-5_l_fore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 scale=0.001 0.001 0.001
- link l_hand: geometry collision mesh filename=package://testbot_description/meshes/dae/sim_sea_2-5_l_hand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 scale=0.001 0.001 0.001; visual mesh filename=package://testbot_description/meshes/dae/sim_sea_2-5_l_hand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 scale=0.001 0.001 0.001
- link l_hip_1: geometry collision mesh filename=package://testbot_description/meshes/dae/sim_sea_2-5_l_hip_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 scale=0.001 0.001 0.001; visual mesh filename=package://testbot_description/meshes/dae/sim_sea_2-5_l_hip_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 scale=0.001 0.001 0.001
- link l_hip_2: geometry collision mesh filename=package://testbot_description/meshes/dae/sim_sea_2-5_l_hip_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 scale=0.001 0.001 0.001; visual mesh filename=package://testbot_description/meshes/dae/sim_sea_2-5_l_hip_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 scale=0.001 0.001 0.001
- link l_hip_3: geometry collision mesh filename=package://testbot_description/meshes/dae/sim_sea_2-5_l_uppe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 scale=0.001 0.001 0.001; visual mesh filename=package://testbot_description/meshes/dae/sim_sea_2-5_l_uppe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 scale=0.001 0.001 0.001
- link l_lower_leg: geometry collision mesh filename=package://testbot_description/meshes/dae/sim_sea_2-5_l_shan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 scale=0.001 0.001 0.001; visual mesh filename=package://testbot_description/meshes/dae/sim_sea_2-5_l_shan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 scale=0.001 0.001 0.001
- link l_shoulder_1: geometry collision mesh filename=package://testbot_description/meshes/dae/sim_sea_2-5_l_shou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 scale=0.001 0.001 0.001; visual mesh filename=package://testbot_description/meshes/dae/sim_sea_2-5_l_shou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 scale=0.001 0.001 0.001
- link l_shoulder_2: geometry collision mesh filename=package://testbot_description/meshes/dae/sim_sea_2-5_l_shou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 scale=0.001 0.001 0.001; visual mesh filename=package://testbot_description/meshes/dae/sim_sea_2-5_l_shou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 scale=0.001 0.001 0.001
- link l_shoulder_3: geometry collision mesh filename=package://testbot_description/meshes/dae/sim_sea_2-5_l_uppe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 scale=0.001 0.001 0.001; visual mesh filename=package://testbot_description/meshes/dae/sim_sea_2-5_l_uppe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 scale=0.001 0.001 0.001
- link l_upper_arm: geometry collision mesh filename=package://testbot_description/meshes/dae/sim_sea_2-5_l_elbo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 scale=0.001 0.001 0.001; visual mesh filename=package://testbot_description/meshes/dae/sim_sea_2-5_l_elbo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 scale=0.001 0.001 0.001
- link l_upper_leg: geometry collision mesh filename=package://testbot_description/meshes/dae/sim_sea_2-5_l_thig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 scale=0.001 0.001 0.001; visual mesh filename=package://testbot_description/meshes/dae/sim_sea_2-5_l_thig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 scale=0.001 0.001 0.001
- link l_wrist_1: geometry collision mesh filename=package://testbot_description/meshes/dae/sim_sea_2-5_l_wris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 scale=0.001 0.001 0.001; visual mesh filename=package://testbot_description/meshes/dae/sim_sea_2-5_l_wris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 scale=0.001 0.001 0.001
- link neck_1: geometry collision mesh filename=package://testbot_description/meshes/dae/sim_sea_2-5_neck_1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 scale=0.001 0.001 0.001; visual mesh filename=package://testbot_description/meshes/dae/sim_sea_2-5_neck_1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 scale=0.001 0.001 0.001
- link neck_2: geometry collision mesh filename=package://testbot_description/meshes/dae/sim_sea_2-5_neck_2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 scale=0.001 0.001 0.001; visual mesh filename=package://testbot_description/meshes/dae/sim_sea_2-5_neck_2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 scale=0.001 0.001 0.001
- link r_ankle_1: geometry collision mesh filename=package://testbot_description/meshes/dae/sim_sea_2-5_r_ankl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 scale=0.001 0.001 0.001; visual mesh filename=package://testbot_description/meshes/dae/sim_sea_2-5_r_ankl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 scale=0.001 0.001 0.001
- link r_ankle_2: geometry collision mesh filename=package://testbot_description/meshes/dae/sim_sea_2-5_r_foot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 scale=0.001 0.001 0.001; visual mesh filename=package://testbot_description/meshes/dae/sim_sea_2-5_r_foot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 scale=0.001 0.001 0.001
- link r_elbow_1: geometry collision mesh filename=package://testbot_description/meshes/dae/sim_sea_2-5_r_elbo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 scale=0.001 0.001 0.001; visual mesh filename=package://testbot_description/meshes/dae/sim_sea_2-5_r_elbo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 scale=0.001 0.001 0.001
- link r_foot: geometry collision mesh filename=package://testbot_description/meshes/dae/sim_sea_2-5_r_sole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 scale=0.001 0.001 0.001; visual mesh filename=package://testbot_description/meshes/dae/sim_sea_2-5_r_sole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 scale=0.001 0.001 0.001
- link r_forearm: geometry collision mesh filename=package://testbot_description/meshes/dae/sim_sea_2-5_r_fore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 scale=0.001 0.001 0.001; visual mesh filename=package://testbot_description/meshes/dae/sim_sea_2-5_r_fore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 scale=0.001 0.001 0.001
- link r_hand: geometry collision mesh filename=package://testbot_description/meshes/dae/sim_sea_2-5_r_hand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 scale=0.001 0.001 0.001; visual mesh filename=package://testbot_description/meshes/dae/sim_sea_2-5_r_hand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 scale=0.001 0.001 0.001
- link r_hip_1: geometry collision mesh filename=package://testbot_description/meshes/dae/sim_sea_2-5_r_hip_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 scale=0.001 0.001 0.001; visual mesh filename=package://testbot_description/meshes/dae/sim_sea_2-5_r_hip_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 scale=0.001 0.001 0.001
- link r_hip_2: geometry collision mesh filename=package://testbot_description/meshes/dae/sim_sea_2-5_r_hip_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 scale=0.001 0.001 0.001; visual mesh filename=package://testbot_description/meshes/dae/sim_sea_2-5_r_hip_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 scale=0.001 0.001 0.001
- link r_hip_3: geometry collision mesh filename=package://testbot_description/meshes/dae/sim_sea_2-5_r_uppe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 scale=0.001 0.001 0.001; visual mesh filename=package://testbot_description/meshes/dae/sim_sea_2-5_r_uppe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 scale=0.001 0.001 0.001
- link r_lower_leg: geometry collision mesh filename=package://testbot_description/meshes/dae/sim_sea_2-5_r_shan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 scale=0.001 0.001 0.001; visual mesh filename=package://testbot_description/meshes/dae/sim_sea_2-5_r_shan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 scale=0.001 0.001 0.001
- link r_shoulder_1: geometry collision mesh filename=package://testbot_description/meshes/dae/sim_sea_2-5_r_shou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 scale=0.001 0.001 0.001; visual mesh filename=package://testbot_description/meshes/dae/sim_sea_2-5_r_shou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 scale=0.001 0.001 0.001
- link r_shoulder_2: geometry collision mesh filename=package://testbot_description/meshes/dae/sim_sea_2-5_r_shou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 scale=0.001 0.001 0.001; visual mesh filename=package://testbot_description/meshes/dae/sim_sea_2-5_r_shou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 scale=0.001 0.001 0.001
- link r_shoulder_3: geometry collision mesh filename=package://testbot_description/meshes/dae/sim_sea_2-5_r_uppe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 scale=0.001 0.001 0.001; visual mesh filename=package://testbot_description/meshes/dae/sim_sea_2-5_r_uppe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 scale=0.001 0.001 0.001
- link r_upper_arm: geometry collision mesh filename=package://testbot_description/meshes/dae/sim_sea_2-5_r_elbo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 scale=0.001 0.001 0.001; visual mesh filename=package://testbot_description/meshes/dae/sim_sea_2-5_r_elbo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 scale=0.001 0.001 0.001
- link r_upper_leg: geometry collision mesh filename=package://testbot_description/meshes/dae/sim_sea_2-5_r_thig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 scale=0.001 0.001 0.001; visual mesh filename=package://testbot_description/meshes/dae/sim_sea_2-5_r_thig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 scale=0.001 0.001 0.001
- link r_wrist_1: geometry collision mesh filename=package://testbot_description/meshes/dae/sim_sea_2-5_r_wris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 scale=0.001 0.001 0.001; visual mesh filename=package://testbot_description/meshes/dae/sim_sea_2-5_r_wris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 scale=0.001 0.001 0.001
- link root_link: geometry collision mesh filename=package://testbot_description/meshes/dae/sim_sea_2-5_root_l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 scale=0.001 0.001 0.001; visual mesh filename=package://testbot_description/meshes/dae/sim_sea_2-5_root_l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 scale=0.001 0.001 0.001
- link torso_1: geometry collision mesh filename=package://testbot_description/meshes/dae/sim_sea_2-5_lap_be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 scale=0.001 0.001 0.001; visual mesh filename=package://testbot_description/meshes/dae/sim_sea_2-5_lap_be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 scale=0.001 0.001 0.001
- link torso_2: geometry collision mesh filename=package://testbot_description/meshes/dae/sim_sea_2-5_lap_be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 scale=0.001 0.001 0.001; visual mesh filename=package://testbot_description/meshes/dae/sim_sea_2-5_lap_be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 scale=0.001 0.001 0.001

File: app/urdfs/iCubGenova04.urdf (robot description, URDF)
Before this commit: robot ICUB_2-5_BB_SIM_MODEL, 163 links, 162 joints
Links:
- link chest: geometry collision mesh filename=package://testbot_description/meshes/dae/sim_sea_2-5_chest_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 scale=0.001 0.001 0.001; visual mesh filename=package://testbot_description/meshes/dae/sim_sea_2-5_chest_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 scale=0.001 0.001 0.001
- link head: geometry collision mesh filename=package://testbot_description/meshes/dae/sim_sea_2-5_head_p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 scale=0.001 0.001 0.001; visual mesh filename=package://testbot_description/meshes/dae/sim_sea_2-5_head_p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 scale=0.001 0.001 0.001
- link l_ankle_1: geometry collision mesh filename=package://testbot_description/meshes/dae/sim_sea_2-5_l_ankl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 scale=0.001 0.001 0.001; visual mesh filename=package://testbot_description/meshes/dae/sim_sea_2-5_l_ankl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 scale=0.001 0.001 0.001
- link l_ankle_2: geometry collision mesh filename=package://testbot_description/meshes/dae/sim_sea_2-5_l_foot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 scale=0.001 0.001 0.001; visual mesh filename=package://testbot_description/meshes/dae/sim_sea_2-5_l_foot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 scale=0.001 0.001 0.001
- link l_elbow_1: geometry collision mesh filename=package://testbot_description/meshes/dae/sim_sea_2-5_l_elbo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 scale=0.001 0.001 0.001; visual mesh filename=package://testbot_description/meshes/dae/sim_sea_2-5_l_elbo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 scale=0.001 0.001 0.001
- link l_foot: geometry collision mesh filename=package://testbot_description/meshes/dae/sim_sea_2-5_l_sole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 scale=0.001 0.001 0.001; visual mesh filename=package://testbot_description/meshes/dae/sim_sea_2-5_l_sole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 scale=0.001 0.001 0.001
- link l_forearm: geometry collision mesh filename=package://testbot_description/meshes/dae/sim_sea_2-5_l_fore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 scale=0.001 0.001 0.001; visual mesh filename=package://testbot_description/meshes/dae/sim_sea_2-5_l_fore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 scale=0.001 0.001 0.001
- link l_hand: geometry collision mesh filename=package://testbot_description/meshes/dae/sim_sea_2-5_l_hand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 scale=0.001 0.001 0.001; visual mesh filename=package://testbot_description/meshes/dae/sim_sea_2-5_l_hand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 scale=0.001 0.001 0.001
- link l_hip_1: geometry collision mesh filename=package://testbot_description/meshes/dae/sim_sea_2-5_l_hip_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 scale=0.001 0.001 0.001; visual mesh filename=package://testbot_description/meshes/dae/sim_sea_2-5_l_hip_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 scale=0.001 0.001 0.001
- link l_hip_2: geometry collision mesh filename=package://testbot_description/meshes/dae/sim_sea_2-5_l_hip_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 scale=0.001 0.001 0.001; visual mesh filename=package://testbot_description/meshes/dae/sim_sea_2-5_l_hip_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 scale=0.001 0.001 0.001
- link l_hip_3: geometry collision mesh filename=package://testbot_description/meshes/dae/sim_sea_2-5_l_uppe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 scale=0.001 0.001 0.001; visual mesh filename=package://testbot_description/meshes/dae/sim_sea_2-5_l_uppe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 scale=0.001 0.001 0.001
- link l_lower_leg: geometry collision mesh filename=package://testbot_description/meshes/dae/sim_sea_2-5_l_shan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 scale=0.001 0.001 0.001; visual mesh filename=package://testbot_description/meshes/dae/sim_sea_2-5_l_shan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 scale=0.001 0.001 0.001
- link l_shoulder_1: geometry collision mesh filename=package://testbot_description/meshes/dae/sim_sea_2-5_l_shou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 scale=0.001 0.001 0.001; visual mesh filename=package://testbot_description/meshes/dae/sim_sea_2-5_l_shou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 scale=0.001 0.001 0.001
- link l_shoulder_2: geometry collision mesh filename=package://testbot_description/meshes/dae/sim_sea_2-5_l_shou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 scale=0.001 0.001 0.001; visual mesh filename=package://testbot_description/meshes/dae/sim_sea_2-5_l_shou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 scale=0.001 0.001 0.001
- link l_shoulder_3: geometry collision mesh filename=package://testbot_description/meshes/dae/sim_sea_2-5_l_uppe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 scale=0.001 0.001 0.001; visual mesh filename=package://testbot_description/meshes/dae/sim_sea_2-5_l_uppe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 scale=0.001 0.001 0.001
- link l_upper_arm: geometry collision mesh filename=package://testbot_description/meshes/dae/sim_sea_2-5_l_elbo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 scale=0.001 0.001 0.001; visual mesh filename=package://testbot_description/meshes/dae/sim_sea_2-5_l_elbo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 scale=0.001 0.001 0.001
- link l_upper_leg: geometry collision mesh filename=package://testbot_description/meshes/dae/sim_sea_2-5_l_thig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 scale=0.001 0.001 0.001; visual mesh filename=package://testbot_description/meshes/dae/sim_sea_2-5_l_thig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 scale=0.001 0.001 0.001
- link l_wrist_1: geometry collision mesh filename=package://testbot_description/meshes/dae/sim_sea_2-5_l_wris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 scale=0.001 0.001 0.001; visual mesh filename=package://testbot_description/meshes/dae/sim_sea_2-5_l_wris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 scale=0.001 0.001 0.001
- link neck_1: geometry collision mesh filename=package://testbot_description/meshes/dae/sim_sea_2-5_neck_1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 scale=0.001 0.001 0.001; visual mesh filename=package://testbot_description/meshes/dae/sim_sea_2-5_neck_1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 scale=0.001 0.001 0.001
- link neck_2: geometry collision mesh filename=package://testbot_description/meshes/dae/sim_sea_2-5_neck_2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 scale=0.001 0.001 0.001; visual mesh filename=package://testbot_description/meshes/dae/sim_sea_2-5_neck_2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 scale=0.001 0.001 0.001
- link r_ankle_1: geometry collision mesh filename=package://testbot_description/meshes/dae/sim_sea_2-5_r_ankl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 scale=0.001 0.001 0.001; visual mesh filename=package://testbot_description/meshes/dae/sim_sea_2-5_r_ankl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 scale=0.001 0.001 0.001
- link r_ankle_2: geometry collision mesh filename=package://testbot_description/meshes/dae/sim_sea_2-5_r_foot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 scale=0.001 0.001 0.001; visual mesh filename=package://testbot_description/meshes/dae/sim_sea_2-5_r_foot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 scale=0.001 0.001 0.001
- link r_elbow_1: geometry collision mesh filename=package://testbot_description/meshes/dae/sim_sea_2-5_r_elbo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 scale=0.001 0.001 0.001; visual mesh filename=package://testbot_description/meshes/dae/sim_sea_2-5_r_elbo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 scale=0.001 0.001 0.001
- link r_foot: geometry collision mesh filename=package://testbot_description/meshes/dae/sim_sea_2-5_r_sole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 scale=0.001 0.001 0.001; visual mesh filename=package://testbot_description/meshes/dae/sim_sea_2-5_r_sole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 scale=0.001 0.001 0.001
- link r_forearm: geometry collision mesh filename=package://testbot_description/meshes/dae/sim_sea_2-5_r_fore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 scale=0.001 0.001 0.001; visual mesh filename=package://testbot_description/meshes/dae/sim_sea_2-5_r_fore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 scale=0.001 0.001 0.001
- link r_hand: geometry collision mesh filename=package://testbot_description/meshes/dae/sim_sea_2-5_r_hand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 scale=0.001 0.001 0.001; visual mesh filename=package://testbot_description/meshes/dae/sim_sea_2-5_r_hand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 scale=0.001 0.001 0.001
- link r_hip_1: geometry collision mesh filename=package://testbot_description/meshes/dae/sim_sea_2-5_r_hip_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 scale=0.001 0.001 0.001; visual mesh filename=package://testbot_description/meshes/dae/sim_sea_2-5_r_hip_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 scale=0.001 0.001 0.001
- link r_hip_2: geometry collision mesh filename=package://testbot_description/meshes/dae/sim_sea_2-5_r_hip_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 scale=0.001 0.001 0.001; visual mesh filename=package://testbot_description/meshes/dae/sim_sea_2-5_r_hip_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 scale=0.001 0.001 0.001
- link r_hip_3: geometry collision mesh filename=package://testbot_description/meshes/dae/sim_sea_2-5_r_uppe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 scale=0.001 0.001 0.001; visual mesh filename=package://testbot_description/meshes/dae/sim_sea_2-5_r_uppe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 scale=0.001 0.001 0.001
- link r_lower_leg: geometry collision mesh filename=package://testbot_description/meshes/dae/sim_sea_2-5_r_shan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 scale=0.001 0.001 0.001; visual mesh filename=package://testbot_description/meshes/dae/sim_sea_2-5_r_shan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 scale=0.001 0.001 0.001
- link r_shoulder_1: geometry collision mesh filename=package://testbot_description/meshes/dae/sim_sea_2-5_r_shou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 scale=0.001 0.001 0.001; visual mesh filename=package://testbot_description/meshes/dae/sim_sea_2-5_r_shou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 scale=0.001 0.001 0.001
- link r_shoulder_2: geometry collision mesh filename=package://testbot_description/meshes/dae/sim_sea_2-5_r_shou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 scale=0.001 0.001 0.001; visual mesh filename=package://testbot_description/meshes/dae/sim_sea_2-5_r_shou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 scale=0.001 0.001 0.001
- link r_shoulder_3: geometry collision mesh filename=package://testbot_description/meshes/dae/sim_sea_2-5_r_uppe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 scale=0.001 0.001 0.001; visual mesh filename=package://testbot_description/meshes/dae/sim_sea_2-5_r_uppe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 scale=0.001 0.001 0.001
- link r_upper_arm: geometry collision mesh filename=package://testbot_description/meshes/dae/sim_sea_2-5_r_elbo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 scale=0.001 0.001 0.001; visual mesh filename=package://testbot_description/meshes/dae/sim_sea_2-5_r_elbo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 scale=0.001 0.001 0.001
- link r_upper_leg: geometry collision mesh filename=package://testbot_description/meshes/dae/sim_sea_2-5_r_thig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 scale=0.001 0.001 0.001; visual mesh filename=package://testbot_description/meshes/dae/sim_sea_2-5_r_thig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 scale=0.001 0.001 0.001
- link r_wrist_1: geometry collision mesh filename=package://testbot_description/meshes/dae/sim_sea_2-5_r_wris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 scale=0.001 0.001 0.001; visual mesh filename=package://testbot_description/meshes/dae/sim_sea_2-5_r_wris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 scale=0.001 0.001 0.001
- link root_link: geometry collision mesh filename=package://testbot_description/meshes/dae/sim_sea_2-5_root_l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 scale=0.001 0.001 0.001; visual mesh filename=package://testbot_description/meshes/dae/sim_sea_2-5_root_l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 scale=0.001 0.001 0.001
- link torso_1: geometry collision mesh filename=package://testbot_description/meshes/dae/sim_sea_2-5_lap_be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 scale=0.001 0.001 0.001; visual mesh filename=package://testbot_description/meshes/dae/sim_sea_2-5_lap_be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 scale=0.001 0.001 0.001
- link torso_2: geometry collision mesh filename=package://testbot_description/meshes/dae/sim_sea_2-5_lap_be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 scale=0.001 0.001 0.001; visual mesh filename=package://testbot_description/meshes/dae/sim_sea_2-5_lap_be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 scale=0.001 0.001 0.001
