Commit message: Add new model with limits

File: app/urdfs/Claudia66DoF_2PILimit.urdf (robot description, URDF)
Before this commit: robot XSensStyleModel_template, 67 links, 66 joints
Joints:
- joint jC1Head_rotx: limit lower=-3.141592 upper=3.141592 effort=30 velocity=1.0 -> lower=-6.283185 upper=6.283185 effort=30 velocity=1.0
- joint jC1Head_roty: limit lower=-3.141592 upper=3.141592 effort=30 velocity=1.0 -> lower=-6.283185 upper=6.283185 effort=30 velocity=1.0
- joint jC1Head_rotz: limit lower=-3.141592 upper=3.141592 effort=30 velocity=1.0 -> lower=-6.283185 upper=6.283185 effort=30 velocity=1.0
- joint jL1T12_rotx: limit lower=-3.141592 upper=3.141592 effort=30 velocity=1.0 -> lower=-6.283185 upper=6.283185 effort=30 velocity=1.0
- joint jL1T12_roty: limit lower=-3.141592 upper=3.141592 effort=30 velocity=1.0 -> lower=-6.283185 upper=6.283185 effort=30 velocity=1.0
- joint jL1T12_rotz: limit lower=-3.141592 upper=3.141592 effort=30 velocity=1.0 -> lower=-6.283185 upper=6.283185 effort=30 velocity=1.0
- joint jL4L3_rotx: limit lower=-3.141592 upper=3.141592 effort=30 velocity=1.0 -> lower=-6.283185 upper=6.283185 effort=30 velocity=1.0
- joint jL4L3_roty: limit lower=-3.141592 upper=3.141592 effort=30 velocity=1.0 -> lower=-6.283185 upper=6.283185 effort=30 velocity=1.0
- joint jL4L3_rotz: limit effort=30 velocity=1.0 -> lower=-6.283185 upper=6.283185 effort=30 velocity=1.0
- joint jL5S1_rotx: limit lower=-3.141592 upper=3.141592 effort=30 velocity=1.0 -> lower=-6.283185 upper=6.283185 effort=30 velocity=1.0
- joint jL5S1_roty: limit lower=-3.141592 upper=3.141592 effort=30 velocity=1.0 -> lower=-6.283185 upper=6.283185 effort=30 velocity=1.0
- joint jL5S1_rotz: limit effort=30 velocity=1.0 -> lower=-6.283185 upper=6.283185 effort=30 velocity=1.0
- joint jLeftAnkle_rotx: limit lower=-3.141592 upper=3.141592 effort=30 velocity=1.0 -> lower=-6.283185 upper=6.283185 effort=30 velocity=1.0
- joint jLeftAnkle_roty: limit lower=-3.141592 upper=3.141592 effort=30 velocity=1.0 -> lower=-6.283185 upper=6.283185 effort=30 velocity=1.0
- joint jLeftAnkle_rotz: limit lower=-3.141592 upper=3.141592 effort=30 velocity=1.0 -> lower=-6.283185 upper=6.283185 effort=30 velocity=1.0
- joint jLeftBallFoot_rotx: limit lower=-3.141592 upper=3.141592 effort=30 velocity=1.0 -> lower=-6.283185 upper=6.283185 effort=30 velocity=1.0
- joint jLeftBallFoot_roty: limit lower=-3.141592 upper=3.141592 effort=30 velocity=1.0 -> lower=-6.283185 upper=6.283185 effort=30 velocity=1.0
- joint jLeftBallFoot_rotz: limit lower=-3.141592 upper=3.141592 effort=30 velocity=1.0 -> lower=-6.283185 upper=6.283185 effort=30 velocity=1.0
- joint jLeftC7Shoulder_rotx: limit lower=-3.141592 upper=3.141592 effort=30 velocity=1.0 -> lower=-6.283185 upper=6.283185 effort=30 velocity=1.0
- joint jLeftC7Shoulder_roty: limit lower=-3.141592 upper=3.141592 effort=30 velocity=1.0 -> lower=-6.283185 upper=6.283185 effort=30 velocity=1.0
- joint jLeftC7Shoulder_rotz: limit lower=-3.141592 upper=3.141592 effort=30 velocity=1.0 -> lower=-6.283185 upper=6.283185 effort=30 velocity=1.0
- joint jLeftElbow_rotx: limit lower=-3.141592 upper=3.141592 effort=30 velocity=1.0 -> lower=-6.283185 upper=6.283185 effort=30 velocity=1.0
- joint jLeftElbow_roty: limit lower=-3.141592 upper=3.141592 effort=30 velocity=1.0 -> lower=-6.283185 upper=6.283185 effort=30 velocity=1.0
- joint jLeftElbow_rotz: limit lower=-3.141592 upper=3.141592 effort=30 velocity=1.0 -> lower=-6.283185 upper=6.283185 effort=30 velocity=1.0
- joint jLeftHip_rotx: limit lower=-3.141592 upper=3.141592 effort=30 velocity=1.0 -> lower=-6.283185 upper=6.283185 effort=30 velocity=1.0
- joint jLeftHip_roty: limit lower=-3.141592 upper=3.141592 effort=30 velocity=1.0 -> lower=-6.283185 upper=6.283185 effort=30 velocity=1.0
- joint jLeftHip_rotz: limit lower=-3.141592 upper=3.141592 effort=30 velocity=1.0 -> lower=-6.283185 upper=6.283185 effort=30 velocity=1.0
- joint jLeftKnee_rotx: limit lower=-3.141592 upper=3.141592 effort=30 velocity=1.0 -> lower=-6.283185 upper=6.283185 effort=30 velocity=1.0
- joint jLeftKnee_roty: limit lower=-3.141592 upper=3.141592 effort=30 velocity=1.0 -> lower=-6.283185 upper=6.283185 effort=30 velocity=1.0
- joint jLeftKnee_rotz: limit lower=-3.141592 upper=3.141592 effort=30 velocity=1.0 -> lower=-6.283185 upper=6.283185 effort=30 velocity=1.0
- joint jLeftShoulder_rotx: limit lower=-3.141592 upper=3.141592 effort=30 velocity=1.0 -> lower=-6.283185 upper=6.283185 effort=30 velocity=1.0
- joint jLeftShoulder_roty: limit lower=-3.141592 upper=3.141592 effort=30 velocity=1.0 -> lower=-6.283185 upper=6.283185 effort=30 velocity=1.0
- joint jLeftShoulder_rotz: limit lower=-3.141592 upper=3.141592 effort=30 velocity=1.0 -> lower=-6.283185 upper=6.283185 effort=30 velocity=1.0
- joint jLeftWrist_rotx: limit lower=-3.141592 upper=3.141592 effort=30 velocity=1.0 -> lower=-6.283185 upper=6.283185 effort=30 velocity=1.0
- joint jLeftWrist_roty: limit lower=-3.141592 upper=3.141592 effort=30 velocity=1.0 -> lower=-6.283185 upper=6.283185 effort=30 velocity=1.0
- joint jLeftWrist_rotz: limit lower=-3.141592 upper=3.141592 effort=30 velocity=1.0 -> lower=-6.283185 upper=6.283185 effort=30 velocity=1.0
- joint jRightAnkle_rotx: limit lower=-3.141592 upper=3.141592 effort=30 velocity=1.0 -> lower=-6.283185 upper=6.283185 effort=30 velocity=1.0
- joint jRightAnkle_roty: limit lower=-3.141592 upper=3.141592 effort=30 velocity=1.0 -> lower=-6.283185 upper=6.283185 effort=30 velocity=1.0
- joint jRightAnkle_rotz: limit lower=-3.141592 upper=3.141592 effort=30 velocity=1.0 -> lower=-6.283185 upper=6.283185 effort=30 velocity=1.0
- joint jRightBallFoot_rotx: limit lower=-3.141592 upper=3.141592 effort=30 velocity=1.0 -> lower=-6.283185 upper=6.283185 effort=30 velocity=1.0
- joint jRightBallFoot_roty: limit lower=-3.141592 upper=3.141592 effort=30 velocity=1.0 -> lower=-6.283185 upper=6.283185 effort=30 velocity=1.0
- joint jRightBallFoot_rotz: limit lower=-3.141592 upper=3.141592 effort=30 velocity=1.0 -> lower=-6.283185 upper=6.283185 effort=30 velocity=1.0
- joint jRightC7Shoulder_rotx: limit lower=-3.141592 upper=3.141592 effort=30 velocity=1.0 -> lower=-6.283185 upper=6.283185 effort=30 velocity=1.0
- joint jRightC7Shoulder_roty: limit lower=-3.141592 upper=3.141592 effort=30 velocity=1.0 -> lower=-6.283185 upper=6.283185 effort=30 velocity=1.0
- joint jRightC7Shoulder_rotz: limit lower=-3.141592 upper=3.141592 effort=30 velocity=1.0 -> lower=-6.283185 upper=6.283185 effort=30 velocity=1.0
- joint jRightElbow_rotx: limit lower=-3.141592 upper=3.141592 effort=30 velocity=1.0 -> lower=-6.283185 upper=6.283185 effort=30 velocity=1.0
- joint jRightElbow_roty: limit lower=-3.141592 upper=3.141592 effort=30 velocity=1.0 -> lower=-6.283185 upper=6.283185 effort=30 velocity=1.0
- joint jRightElbow_rotz: limit lower=-3.141592 upper=3.141592 effort=30 velocity=1.0 -> lower=-6.283185 upper=6.283185 effort=30 velocity=1.0
- joint jRightHip_rotx: limit lower=-3.141592 upper=3.141592 effort=30 velocity=1.0 -> lower=-6.283185 upper=6.283185 effort=30 velocity=1.0
- joint jRightHip_roty: limit lower=-3.141592 upper=3.141592 effort=30 velocity=1.0 -> lower=-6.283185 upper=6.283185 effort=30 velocity=1.0
- joint jRightHip_rotz: limit lower=-3.141592 upper=3.141592 effort=30 velocity=1.0 -> lower=-6.283185 upper=6.283185 effort=30 velocity=1.0
- joint jRightKnee_rotx: limit lower=-3.141592 upper=3.141592 effort=30 velocity=1.0 -> lower=-6.283185 upper=6.283185 effort=30 velocity=1.0
- joint jRightKnee_roty: limit lower=-3.141592 upper=3.141592 effort=30 velocity=1.0 -> lower=-6.283185 upper=6.283185 effort=30 velocity=1.0
- joint jRightKnee_rotz: limit lower=-3.141592 upper=3.141592 effort=30 velocity=1.0 -> lower=-6.283185 upper=6.283185 effort=30 velocity=1.0
- joint jRightShoulder_rotx: limit lower=-3.141592 upper=3.141592 effort=30 velocity=1.0 -> lower=-6.283185 upper=6.283185 effort=30 velocity=1.0
- joint jRightShoulder_roty: limit lower=-3.141592 upper=3.141592 effort=30 velocity=1.0 -> lower=-6.283185 upper=6.283185 effort=30 velocity=1.0
- joint jRightShoulder_rotz: limit lower=-3.141592 upper=3.141592 effort=30 velocity=1.0 -> lower=-6.283185 upper=6.283185 effort=30 velocity=1.0
- joint jRightWrist_rotx: limit lower=-3.141592 upper=3.141592 effort=30 velocity=1.0 -> lower=-6.283185 upper=6.283185 effort=30 velocity=1.0
- joint jRightWrist_roty: limit lower=-3.141592 upper=3.141592 effort=30 velocity=1.0 -> lower=-6.283185 upper=6.283185 effort=30 velocity=1.0
- joint jRightWrist_rotz: limit lower=-3.141592 upper=3.141592 effort=30 velocity=1.0 -> lower=-6.283185 upper=6.283185 effort=30 velocity=1.0
- joint jT1C7_rotx: limit lower=-3.141592 upper=3.141592 effort=30 velocity=1.0 -> lower=-6.283185 upper=6.283185 effort=30 velocity=1.0
- joint jT1C7_roty: limit lower=-3.141592 upper=3.141592 effort=30 velocity=1.0 -> lower=-6.283185 upper=6.283185 effort=30 velocity=1.0
- joint jT1C7_rotz: limit lower=-3.141592 upper=3.141592 effort=30 velocity=1.0 -> lower=-6.283185 upper=6.283185 effort=30 velocity=1.0
- joint jT9T8_rotx: limit lower=-3.141592 upper=3.141592 effort=30 velocity=1.0 -> lower=-6.283185 upper=6.283185 effort=30 velocity=1.0
- joint jT9T8_roty: limit lower=-3.141592 upper=3.141592 effort=30 velocity=1.0 -> lower=-6.283185 upper=6.283185 effort=30 velocity=1.0
- joint jT9T8_rotz: limit lower=-3.141592 upper=3.141592 effort=30 velocity=1.0 -> lower=-6.283185 upper=6.283185 effort=30 velocity=1.0

File: app/urdfs/Claudia66DoF_PILimit.urdf (robot description, URDF)
Before this commit: robot XSensStyleModel_template, 67 links, 66 joints
Joints:
- joint jL4L3_rotz: limit effort=30 velocity=1.0 -> lower=-3.141592 upper=3.141592 effort=30 velocity=1.0
- joint jL5S1_rotz: limit effort=30 velocity=1.0 -> lower=-3.141592 upper=3.141592 effort=30 velocity=1.0

File: app/urdfs/Claudia66DoF_e16Limit.urdf (robot description, URDF)
Before this commit: robot XSensStyleModel_template, 67 links, 66 joints
Joints:
- joint jC1Head_rotx: limit lower=-3.141592 upper=3.141592 effort=30 velocity=1.0 -> lower=-1e+16 upper=1e+16 effort=30 velocity=1.0
- joint jC1Head_roty: limit lower=-3.141592 upper=3.141592 effort=30 velocity=1.0 -> lower=-1e+16 upper=1e+16 effort=30 velocity=1.0
- joint jC1Head_rotz: limit lower=-3.141592 upper=3.141592 effort=30 velocity=1.0 -> lower=-1e+16 upper=1e+16 effort=30 velocity=1.0
- joint jL1T12_rotx: limit lower=-3.141592 upper=3.141592 effort=30 velocity=1.0 -> lower=-1e+16 upper=1e+16 effort=30 velocity=1.0
- joint jL1T12_roty: limit lower=-3.141592 upper=3.141592 effort=30 velocity=1.0 -> lower=-1e+16 upper=1e+16 effort=30 velocity=1.0
- joint jL1T12_rotz: limit lower=-3.141592 upper=3.141592 effort=30 velocity=1.0 -> lower=-1e+16 upper=1e+16 effort=30 velocity=1.0
- joint jL4L3_rotx: limit lower=-3.141592 upper=3.141592 effort=30 velocity=1.0 -> lower=-1e+16 upper=1e+16 effort=30 velocity=1.0
- joint jL4L3_roty: limit lower=-3.141592 upper=3.141592 effort=30 velocity=1.0 -> lower=-1e+16 upper=1e+16 effort=30 velocity=1.0
- joint jL4L3_rotz: limit effort=30 velocity=1.0 -> lower=-1e+16 upper=1e+16 effort=30 velocity=1.0
- joint jL5S1_rotx: limit lower=-3.141592 upper=3.141592 effort=30 velocity=1.0 -> lower=-1e+16 upper=1e+16 effort=30 velocity=1.0
- joint jL5S1_roty: limit lower=-3.141592 upper=3.141592 effort=30 velocity=1.0 -> lower=-1e+16 upper=1e+16 effort=30 velocity=1.0
- joint jL5S1_rotz: limit effort=30 velocity=1.0 -> lower=-1e+16 upper=1e+16 effort=30 velocity=1.0
- joint jLeftAnkle_rotx: limit lower=-3.141592 upper=3.141592 effort=30 velocity=1.0 -> lower=-1e+16 upper=1e+16 effort=30 velocity=1.0
- joint jLeftAnkle_roty: limit lower=-3.141592 upper=3.141592 effort=30 velocity=1.0 -> lower=-1e+16 upper=1e+16 effort=30 velocity=1.0
- joint jLeftAnkle_rotz: limit lower=-3.141592 upper=3.141592 effort=30 velocity=1.0 -> lower=-1e+16 upper=1e+16 effort=30 velocity=1.0
- joint jLeftBallFoot_rotx: limit lower=-3.141592 upper=3.141592 effort=30 velocity=1.0 -> lower=-1e+16 upper=1e+16 effort=30 velocity=1.0
- joint jLeftBallFoot_roty: limit lower=-3.141592 upper=3.141592 effort=30 velocity=1.0 -> lower=-1e+16 upper=1e+16 effort=30 velocity=1.0
- joint jLeftBallFoot_rotz: limit lower=-3.141592 upper=3.141592 effort=30 velocity=1.0 -> lower=-1e+16 upper=1e+16 effort=30 velocity=1.0
- joint jLeftC7Shoulder_rotx: limit lower=-3.141592 upper=3.141592 effort=30 velocity=1.0 -> lower=-1e+16 upper=1e+16 effort=30 velocity=1.0
- joint jLeftC7Shoulder_roty: limit lower=-3.141592 upper=3.141592 effort=30 velocity=1.0 -> lower=-1e+16 upper=1e+16 effort=30 velocity=1.0
- joint jLeftC7Shoulder_rotz: limit lower=-3.141592 upper=3.141592 effort=30 velocity=1.0 -> lower=-1e+16 upper=1e+16 effort=30 velocity=1.0
- joint jLeftElbow_rotx: limit lower=-3.141592 upper=3.141592 effort=30 velocity=1.0 -> lower=-1e+16 upper=1e+16 effort=30 velocity=1.0
- joint jLeftElbow_roty: limit lower=-3.141592 upper=3.141592 effort=30 velocity=1.0 -> lower=-1e+16 upper=1e+16 effort=30 velocity=1.0
- joint jLeftElbow_rotz: limit lower=-3.141592 upper=3.141592 effort=30 velocity=1.0 -> lower=-1e+16 upper=1e+16 effort=30 velocity=1.0
- joint jLeftHip_rotx: limit lower=-3.141592 upper=3.141592 effort=30 velocity=1.0 -> lower=-1e+16 upper=1e+16 effort=30 velocity=1.0
- joint jLeftHip_roty: limit lower=-3.141592 upper=3.141592 effort=30 velocity=1.0 -> lower=-1e+16 upper=1e+16 effort=30 velocity=1.0
- joint jLeftHip_rotz: limit lower=-3.141592 upper=3.141592 effort=30 velocity=1.0 -> lower=-1e+16 upper=1e+16 effort=30 velocity=1.0
- joint jLeftKnee_rotx: limit lower=-3.141592 upper=3.141592 effort=30 velocity=1.0 -> lower=-1e+16 upper=1e+16 effort=30 velocity=1.0
- joint jLeftKnee_roty: limit lower=-3.141592 upper=3.141592 effort=30 velocity=1.0 -> lower=-1e+16 upper=1e+16 effort=30 velocity=1.0
- joint jLeftKnee_rotz: limit lower=-3.141592 upper=3.141592 effort=30 velocity=1.0 -> lower=-1e+16 upper=1e+16 effort=30 velocity=1.0
- joint jLeftShoulder_rotx: limit lower=-3.141592 upper=3.141592 effort=30 velocity=1.0 -> lower=-1e+16 upper=1e+16 effort=30 velocity=1.0
- joint jLeftShoulder_roty: limit lower=-3.141592 upper=3.141592 effort=30 velocity=1.0 -> lower=-1e+16 upper=1e+16 effort=30 velocity=1.0
- joint jLeftShoulder_rotz: limit lower=-3.141592 upper=3.141592 effort=30 velocity=1.0 -> lower=-1e+16 upper=1e+16 effort=30 velocity=1.0
- joint jLeftWrist_rotx: limit lower=-3.141592 upper=3.141592 effort=30 velocity=1.0 -> lower=-1e+16 upper=1e+16 effort=30 velocity=1.0
- joint jLeftWrist_roty: limit lower=-3.141592 upper=3.141592 effort=30 velocity=1.0 -> lower=-1e+16 upper=1e+16 effort=30 velocity=1.0
- joint jLeftWrist_rotz: limit lower=-3.141592 upper=3.141592 effort=30 velocity=1.0 -> lower=-1e+16 upper=1e+16 effort=30 velocity=1.0
- joint jRightAnkle_rotx: limit lower=-3.141592 upper=3.141592 effort=30 velocity=1.0 -> lower=-1e+16 upper=1e+16 effort=30 velocity=1.0
- joint jRightAnkle_roty: limit lower=-3.141592 upper=3.141592 effort=30 velocity=1.0 -> lower=-1e+16 upper=1e+16 effort=30 velocity=1.0
- joint jRightAnkle_rotz: limit lower=-3.141592 upper=3.141592 effort=30 velocity=1.0 -> lower=-1e+16 upper=1e+16 effort=30 velocity=1.0
- joint jRightBallFoot_rotx: limit lower=-3.141592 upper=3.141592 effort=30 velocity=1.0 -> lower=-1e+16 upper=1e+16 effort=30 velocity=1.0
- joint jRightBallFoot_roty: limit lower=-3.141592 upper=3.141592 effort=30 velocity=1.0 -> lower=-1e+16 upper=1e+16 effort=30 velocity=1.0
- joint jRightBallFoot_rotz: limit lower=-3.141592 upper=3.141592 effort=30 velocity=1.0 -> lower=-1e+16 upper=1e+16 effort=30 velocity=1.0
- joint jRightC7Shoulder_rotx: limit lower=-3.141592 upper=3.141592 effort=30 velocity=1.0 -> lower=-1e+16 upper=1e+16 effort=30 velocity=1.0
- joint jRightC7Shoulder_roty: limit lower=-3.141592 upper=3.141592 effort=30 velocity=1.0 -> lower=-1e+16 upper=1e+16 effort=30 velocity=1.0
- joint jRightC7Shoulder_rotz: limit lower=-3.141592 upper=3.141592 effort=30 velocity=1.0 -> lower=-1e+16 upper=1e+16 effort=30 velocity=1.0
- joint jRightElbow_rotx: limit lower=-3.141592 upper=3.141592 effort=30 velocity=1.0 -> lower=-1e+16 upper=1e+16 effort=30 velocity=1.0
- joint jRightElbow_roty: limit lower=-3.141592 upper=3.141592 effort=30 velocity=1.0 -> lower=-1e+16 upper=1e+16 effort=30 velocity=1.0
- joint jRightElbow_rotz: limit lower=-3.141592 upper=3.141592 effort=30 velocity=1.0 -> lower=-1e+16 upper=1e+16 effort=30 velocity=1.0
- joint jRightHip_rotx: limit lower=-3.141592 upper=3.141592 effort=30 velocity=1.0 -> lower=-1e+16 upper=1e+16 effort=30 velocity=1.0
- joint jRightHip_roty: limit lower=-3.141592 upper=3.141592 effort=30 velocity=1.0 -> lower=-1e+16 upper=1e+16 effort=30 velocity=1.0
- joint jRightHip_rotz: limit lower=-3.141592 upper=3.141592 effort=30 velocity=1.0 -> lower=-1e+16 upper=1e+16 effort=30 velocity=1.0
- joint jRightKnee_rotx: limit lower=-3.141592 upper=3.141592 effort=30 velocity=1.0 -> lower=-1e+16 upper=1e+16 effort=30 velocity=1.0
- joint jRightKnee_roty: limit lower=-3.141592 upper=3.141592 effort=30 velocity=1.0 -> lower=-1e+16 upper=1e+16 effort=30 velocity=1.0
- joint jRightKnee_rotz: limit lower=-3.141592 upper=3.141592 effort=30 velocity=1.0 -> lower=-1e+16 upper=1e+16 effort=30 velocity=1.0
- joint jRightShoulder_rotx: limit lower=-3.141592 upper=3.141592 effort=30 velocity=1.0 -> lower=-1e+16 upper=1e+16 effort=30 velocity=1.0
- joint jRightShoulder_roty: limit lower=-3.141592 upper=3.141592 effort=30 velocity=1.0 -> lower=-1e+16 upper=1e+16 effort=30 velocity=1.0
- joint jRightShoulder_rotz: limit lower=-3.141592 upper=3.141592 effort=30 velocity=1.0 -> lower=-1e+16 upper=1e+16 effort=30 velocity=1.0
- joint jRightWrist_rotx: limit lower=-3.141592 upper=3.141592 effort=30 velocity=1.0 -> lower=-1e+16 upper=1e+16 effort=30 velocity=1.0
- joint jRightWrist_roty: limit lower=-3.141592 upper=3.141592 effort=30 velocity=1.0 -> lower=-1e+16 upper=1e+16 effort=30 velocity=1.0
- joint jRightWrist_rotz: limit lower=-3.141592 upper=3.141592 effort=30 velocity=1.0 -> lower=-1e+16 upper=1e+16 effort=30 velocity=1.0
- joint jT1C7_rotx: limit lower=-3.141592 upper=3.141592 effort=30 velocity=1.0 -> lower=-1e+16 upper=1e+16 effort=30 velocity=1.0
- joint jT1C7_roty: limit lower=-3.141592 upper=3.141592 effort=30 velocity=1.0 -> lower=-1e+16 upper=1e+16 effort=30 velocity=1.0
- joint jT1C7_rotz: limit lower=-3.141592 upper=3.141592 effort=30 velocity=1.0 -> lower=-1e+16 upper=1e+16 effort=30 velocity=1.0
- joint jT9T8_rotx: limit lower=-3.141592 upper=3.141592 effort=30 velocity=1.0 -> lower=-1e+16 upper=1e+16 effort=30 velocity=1.0
- joint jT9T8_roty: limit lower=-3.141592 upper=3.141592 effort=30 velocity=1.0 -> lower=-1e+16 upper=1e+16 effort=30 velocity=1.0
- joint jT9T8_rotz: limit lower=-3.141592 upper=3.141592 effort=30 velocity=1.0 -> lower=-1e+16 upper=1e+16 effort=30 velocity=1.0
