Commit message: add fake links to the urdf of the icub

File: app/icubTeleoperationModels/teleoperation_iCub_model_V_2_5/model.urdf (robot description, URDF)
Before this commit: robot iCub, 191 links, 190 joints
Links:
- added link head_fake, mass 0.00001; visual box size=0.2 0.1 0.05
- link chest_fake: mass 0.00001 -> None; geometry 
Joints:
- added joint j_head_fake: type revolute, parent head, child head_fake, origin xyz=0.01 0.01 0.01 rpy=-1.57079632679 -1.57079632679 0, axis 1 0 0, limit lower=-3.141592 upper=3.141592 effort=30 velocity=1.0
- joint j_chest_fake: axis 1 0 0 -> 0 0 0; limit lower=-3.141592 upper=3.141592 effort=30 velocity=1.0 -> (none); origin xyz=0.01 0.01 0.01 rpy=1.57079632679 0 1.57079632679 -> xyz=0 0 0 rpy=-1.57079632679 -1.57079632679 0; type revolute -> fixed
- joint j_root_link_fake: axis 1 0 0 -> 0 0 0

Commit message: add fake links for the icub for the Xsens (some of the fake links have not correct orientation )

File: app/icubTeleoperationModels/teleoperation_iCub_model_V_2_5/model.urdf (robot description, URDF)
Before this commit: robot iCub, 192 links, 191 joints
Links:
- link head_fake: mass 0.00001 -> None; geometry 
Joints:
- joint j_head_fake: axis 1 0 0 -> 0 0 0; limit lower=-3.141592 upper=3.141592 effort=30 velocity=1.0 -> (none); origin xyz=0.01 0.01 0.01 rpy=-1.57079632679 -1.57079632679 0 -> xyz=0 0 0 rpy=-1.57079632679 -1.57079632679 0; type revolute -> fixed
