Commit message: modified 1- the icub model for the fake links, 2- the initial value of the IK solver is the mean of the joint limits

File: app/icubTeleoperationModels/teleoperation_iCub_model_V_2_5/teleoperation_iCub_model_V_2_5.urdf (robot description, URDF)
Before this commit: robot iCub, 204 links, 203 joints
Joints:
- joint j_l_forearm_fake: origin xyz=0 0 0 rpy=0 -1.57079632679 0 -> xyz=0 0 0 rpy=-1.57079632679 -1.57079632679 0
- joint j_l_hand_fake: origin xyz=0 0 0 rpy=0 -1.57079632679 0 -> xyz=0 0 0 rpy=-1.57079632679 -1.57079632679 0
- joint j_l_upper_arm_fake: origin xyz=0 0 0 rpy=3.14159 0 0 -> xyz=0 0 0 rpy=1.57079632679 0 0
- joint j_r_forearm_fake: origin xyz=0 0 0 rpy=3.14159 -1.57079632679 0 -> xyz=0 0 0 rpy=-1.57079632679 -1.57079632679 0
- joint j_r_hand_fake: origin xyz=0 0 0 rpy=3.14159 -1.57079632679 0 -> xyz=0 0 0 rpy=-1.57079632679 -1.57079632679 0
- joint j_r_upper_arm_fake: origin xyz=0 0 0 rpy=3.14159 0 0 -> xyz=0 0 0 rpy=-1.57079632679 0 0

Commit message: change the rate of wrapper, optmazation threshold, initial value of the optimization

File: app/icubTeleoperationModels/teleoperation_iCub_model_V_2_5/teleoperation_iCub_model_V_2_5.urdf (robot description, URDF)
Before this commit: robot iCub, 204 links, 203 joints
Joints:
- joint l_shoulder_roll: limit lower=0.0 upper=2.80648943721 effort=50000 velocity=50000 -> lower=0.35 upper=2.80648943721 effort=50000 velocity=50000
- joint r_shoulder_roll: limit lower=0.0 upper=2.80648943721 effort=50000 velocity=50000 -> lower=0.35 upper=2.80648943721 effort=50000 velocity=50000

Commit message: IROS 2019 code version

File: app/icubTeleoperationModels/teleoperation_iCub_model_V_2_5/teleoperation_iCub_model_V_2_5.urdf (robot description, URDF)
Before this commit: robot iCub, 204 links, 203 joints
Joints:
- joint l_hip_roll: limit lower=-0.349065850399 upper=2.09439510239 effort=37.0 velocity=7.64 -> lower=0.261799000003794 upper=2.09439510239 effort=37.0 velocity=7.64
- joint r_hip_roll: limit lower=-0.349065850399 upper=2.09439510239 effort=37.0 velocity=7.64 -> lower=0.261799000003794 upper=2.09439510239 effort=37.0 velocity=7.64
