Commit message: update configuration and fix pairwised initialization

File: conf/urdfs/teleoperation_iCub_model_V_2_5.urdf (robot description, URDF)
Before this commit: robot iCub, 204 links, 203 joints
Joints:
- joint l_hip_roll: limit lower=0.261799000003794 upper=2.09439510239 effort=37.0 velocity=7.64 -> lower=-0.349065850399 upper=2.09439510239 effort=37.0 velocity=7.64
- joint r_hip_roll: limit lower=0.261799000003794 upper=2.09439510239 effort=37.0 velocity=7.64 -> lower=-0.349065850399 upper=2.09439510239 effort=37.0 velocity=7.64
