Commit message: fix the wrong neck joint axis
Update XsensRetargetingPositionControlPoleiCub3.xml

File: conf/urdfs/teleoperation_iCub_model_V_3.urdf (robot description, URDF)
Before this commit: robot iCub, 54 links, 53 joints
Joints:
- joint neck_yaw: axis 1.6255499221370677e-21 1.0999983743979075e-15 -1.0 -> 1.6255499221370677e-21 1.0999983743979075e-15 1.0

Commit message: Fix r_wrist_yaw joint type and limits

File: conf/urdfs/teleoperation_iCub_model_V_3.urdf (robot description, URDF)
Before this commit: robot iCub, 54 links, 53 joints
Joints:
- joint r_wrist_yaw: limit (none) -> lower=-0.2617993877991494 upper=0.6108652381980153 effort=50000 velocity=120.0; type continuous -> revolute

Commit message: add the xml and urdf for the senseGlove running

File: conf/urdfs/teleoperation_iCub_model_V_3.urdf (robot description, URDF)
Before this commit: robot iCub, 54 links, 53 joints
Links:
- added link l_hand_fake_sg, mass 0.0001
- added link r_hand_fake_sg, mass 0.0001
Joints:
- added joint j_l_hand_fake_sg: type fixed, parent l_hand, child l_hand_fake_sg, origin xyz=0 0 0 rpy=-1.57079632679 0 1.57079632679, axis 0 0 0
- added joint j_r_hand_fake_sg: type fixed, parent r_hand, child r_hand_fake_sg, origin xyz=0 0 0 rpy=1.57079632679 0 -1.57079632679, axis 0 0 0

Commit message: fix the urdf for senseGlove transformation  and bad closing of IK

File: conf/urdfs/teleoperation_iCub_model_V_3.urdf (robot description, URDF)
Before this commit: robot iCub, 56 links, 55 joints
Joints:
- joint j_l_hand_fake_sg: origin xyz=0 0 0 rpy=-1.57079632679 0 1.57079632679 -> xyz=0 0 0 rpy=-1.57079632679 1.57079632679 0
- joint j_r_hand_fake_sg: origin xyz=0 0 0 rpy=1.57079632679 0 -1.57079632679 -> xyz=0 0 0 rpy=1.57079632679 1.57079632679 0

Commit message: Add sense glove changes to include it in IK (#258)
* add the xml and urdf for the senseGlove running

* fix the urdf for senseGlove transformation  and bad closing of IK

* update icub3 retargeting using XSens and SenseGlove; add iFeel SenseGlove Retargeting yarprobotinterface config file

* --amend

* --amend

File: conf/urdfs/teleoperation_iCub_model_V_3.urdf (robot description, URDF)
Before this commit: robot iCub, 54 links, 53 joints
Links:
- added link l_hand_fake_sg, mass 0.0001
- added link r_hand_fake_sg, mass 0.0001
Joints:
- added joint j_l_hand_fake_sg: type fixed, parent l_hand, child l_hand_fake_sg, origin xyz=0 0 0 rpy=-1.57079632679 1.57079632679 0, axis 0 0 0
- added joint j_r_hand_fake_sg: type fixed, parent r_hand, child r_hand_fake_sg, origin xyz=0 0 0 rpy=1.57079632679 1.57079632679 0, axis 0 0 0

Commit message: update the icub3 urdf model elbow joints limits to have a higher range of motion

File: conf/urdfs/teleoperation_iCub_model_V_3.urdf (robot description, URDF)
Before this commit: robot iCub, 56 links, 55 joints
Joints:
- joint l_elbow: limit lower=-0.05235987755982989 upper=1.3089969389957472 effort=50000 velocity=120.0 -> lower=0.0 upper=1.832595714594046 effort=50000 velocity=120.0
- joint r_elbow: limit lower=-0.05235987755982989 upper=1.3089969389957472 effort=50000 velocity=120.0 -> lower=0.0 upper=1.832595714594046 effort=50000 velocity=120.0

Commit message: Update neck joint limits

File: conf/urdfs/teleoperation_iCub_model_V_3.urdf (robot description, URDF)
Before this commit: robot iCub, 56 links, 55 joints
Joints:
- joint neck_pitch: limit lower=-0.5235987755982988 upper=0.3839724354387525 effort=50000 velocity=120.0 -> lower=-0.698132 upper=0.3839724354387525 effort=50000 velocity=120.0

Commit message: Update configuration files

File: conf/urdfs/teleoperation_iCub_model_V_3.urdf (robot description, URDF)
Before this commit: robot iCub, 56 links, 55 joints
Joints:
- joint l_shoulder_pitch: limit lower=-1.53588974175501 upper=0.22689280275926285 effort=50000 velocity=120.0 -> lower=-3.14 upper=0.43 effort=50000 velocity=120.0
- joint r_shoulder_pitch: limit lower=-1.53588974175501 upper=0.22689280275926285 effort=50000 velocity=120.0 -> lower=-3.14 upper=0.43 effort=50000 velocity=120.0

Commit message: [teleoperation_iCub_model_V_3] Uptdate the shoulder_pitch upper limits accordingly to robotology/robots-configuration@51b36db82171e5bf377170cb7c0802ef6e2c30c9

File: conf/urdfs/teleoperation_iCub_model_V_3.urdf (robot description, URDF)
Before this commit: robot iCub, 56 links, 55 joints
Joints:
- joint l_shoulder_pitch: limit lower=-3.14 upper=0.43 effort=50000 velocity=120.0 -> lower=-3.14 upper=0.34 effort=50000 velocity=120.0
- joint r_shoulder_pitch: limit lower=-3.14 upper=0.43 effort=50000 velocity=120.0 -> lower=-3.14 upper=0.34 effort=50000 velocity=120.0

Commit message: [teleoperation_iCub_model_V_3] Uptdate the shoulder_pitch lower limits accordingly to robotology/robots-configuration@51b36db
Co-authored-by: Lorenzo Rapetti <lor.rapetti@gmail.com>

File: conf/urdfs/teleoperation_iCub_model_V_3.urdf (robot description, URDF)
Before this commit: robot iCub, 56 links, 55 joints
Joints:
- joint l_shoulder_pitch: limit lower=-3.14 upper=0.34 effort=50000 velocity=120.0 -> lower=-3.05 upper=0.34 effort=50000 velocity=120.0
- joint r_shoulder_pitch: limit lower=-3.14 upper=0.34 effort=50000 velocity=120.0 -> lower=-3.05 upper=0.34 effort=50000 velocity=120.0
